Commit message: Added the Lidar link/joint

File: description/robot.urdf.xacro (robot description, xacro)
@@ -3,3 +3,5 @@
     <xacro:include filename="$(find wally_boxxy)/description/common_propreties.xacro" />
     <xacro:include filename="$(find wally_boxxy)/description/robot_core.xacro" />
+    <xacro:include filename="$(find wally_boxxy)/description/gazebo_control.xacro" />
+    <xacro:include filename="$(find wally_boxxy)/description/lidar.xacro" />
 </robot>

File: description/robot_core.xacro (robot description, xacro)
@@ -5,5 +5,5 @@
     <link name="chassis">
         <visual>
-            <origin xyz="0.3 0 0.1" rpy="0 0 0" />
+            <origin xyz="0.3 0 0.135" rpy="0 0 0" />
             <geometry>
                 <box size="0.6 0.4 0.2" />
@@ -29,5 +29,5 @@
             <origin xyz="0 0 0" rpy="0 0 0" />
             <geometry>
-                <cylinder length="0.05" radius="0.1" />
+                <cylinder length="0.04" radius="0.055" />
             </geometry>
             <material name="purple" />
@@ -36,8 +36,8 @@
             <origin xyz="0 0 0" rpy="0 0 0" />
             <geometry>
-                <cylinder length="0.05" radius="0.1" />
+                <cylinder length="0.04" radius="0.055" />
             </geometry>
         </collision>
-        <xacro:cylinder_inertia m="0.1" r="0.1" l="0.05" o_xyz="0 0 0" o_rpy="0 0 0" />
+        <xacro:cylinder_inertia m="0.1" r="0.055" l="0.04" o_xyz="0 0 0" o_rpy="0 0 0" />
     </link>
     <joint name="right_wheel_joint" type="continuous">
@@ -51,5 +51,5 @@
             <origin xyz="0 0 0" rpy="0 0 0" />
             <geometry>
-                <cylinder length="0.05" radius="0.1" />
+                <cylinder length="0.04" radius="0.055" />
             </geometry>
         </visual>
@@ -57,8 +57,8 @@
             <origin xyz="0 0 0" rpy="0 0 0" />
             <geometry>
-                <cylinder length="0.05" radius="0.1" />
+                <cylinder length="0.04" radius="0.055" />
             </geometry>
         </collision>
-        <xacro:cylinder_inertia m="0.1" r="0.1" l="0.05" o_xyz="0 0 0" o_rpy="0 0 0" />
+        <xacro:cylinder_inertia m="0.1" r="0.055" l="0.04" o_xyz="0 0 0" o_rpy="0 0 0" />
     </link>
     <joint name="base_link_joint" type="fixed">
