Commit message: RViz2 working, plugins working, Gazebo working, robot model working, bridge working. This is the first commit of the project, with all the files that were created during the development process. The only file that was deleted is the empty world file, which is no longer needed since we have a custom world for testing.

File: description/gazebo_control.xacro (robot description, xacro)
@@ -1,5 +1,5 @@
 <?xml version="1.0"?>
 <robot xmlns:xacro="http://www.ros.org/wiki/xacro">
-    <gazebo>
+    <!-- <gazebo>
         <plugin name="diff_drive" filename="libgazebo_ros_diff_drive.so">
             <left_joint>left_wheel_joint</left_joint>
@@ -16,4 +16,28 @@
             <publish_wheel_tf>true</publish_wheel_tf>
         </plugin>
+    </gazebo> -->
+    <gazebo reference="castor_wheel_link">
+        <mu1 value="0.1" />
+        <mu2 value="0.1" />
+    </gazebo>
+    <gazebo>
+        <plugin
+            filename="gz-sim-diff-drive-system"
+            name="gz::sim::systems::DiffDrive">
+            <left_joint>left_wheel_joint</left_joint>
+            <right_joint>right_wheel_joint</right_joint>
+            <wheel_separation>0.44</wheel_separation>
+            <wheel_radius>0.055</wheel_radius>
+            <frame_id>odom</frame_id>
+            <child_frame_id>base_link</child_frame_id>
+        </plugin>
+    </gazebo>
+    <gazebo>
+        <plugin
+            filename="gz-sim-joint-state-publisher-system"
+            name="gz::sim::systems::JointStatePublisher">
+            <joint_name>left_wheel_joint</joint_name>
+            <joint_name>right_wheel_joint</joint_name>
+        </plugin>
     </gazebo>
 </robot>

File: description/lidar.xacro (robot description, xacro)
@@ -8,5 +8,5 @@
     <link name="laser_link">
         <visual>
-            <origin xyz="0 0 0.05" rpy="0 0 0" />
+            <origin xyz="0 0 0.025" rpy="0 0 0" />
             <geometry>
                 <cylinder length="0.05" radius="0.05" />

File: description/robot_core.xacro (robot description, xacro)
@@ -3,7 +3,12 @@
     <link name="base_link">
     </link>
+    <joint name="base_link_joint" type="fixed">
+        <parent link="base_link" />
+        <child link="chassis" />
+        <origin xyz="-0.3 0 0.035" rpy="0 0 0" />
+    </joint>
     <link name="chassis">
         <visual>
-            <origin xyz="0.3 0 0.135" rpy="0 0 0" />
+            <origin xyz="0.3 0 0.1" rpy="0 0 0" />
             <geometry>
                 <box size="0.6 0.4 0.2" />
@@ -20,7 +25,7 @@
     </link>
     <joint name="left_wheel_joint" type="continuous">
-        <parent link="base_link" />
+        <parent link="chassis" />
         <child link="left_wheel" />
-        <origin xyz="0 0.225 0" rpy="-${pi/2} 0 0" />
+        <origin xyz="0.1 0.22 0.02" rpy="-${pi/2} 0 0" />
         <axis xyz="0 0 1" />
     </joint>
@@ -42,7 +47,7 @@
     </link>
     <joint name="right_wheel_joint" type="continuous">
-        <parent link="base_link" />
+        <parent link="chassis" />
         <child link="right_wheel" />
-        <origin xyz="0 -0.225 0" rpy="${pi/2} 0 0" />
+        <origin xyz="0.1 -0.22 0.02" rpy="${pi/2} 0 0" />
         <axis xyz="0 0 1" />
     </joint>
@@ -53,4 +58,5 @@
                 <cylinder length="0.04" radius="0.055" />
             </geometry>
+            <material name="purple" />
         </visual>
         <collision>
@@ -62,9 +68,4 @@
         <xacro:cylinder_inertia m="0.1" r="0.055" l="0.04" o_xyz="0 0 0" o_rpy="0 0 0" />
     </link>
-    <joint name="base_link_joint" type="fixed">
-        <parent link="base_link" />
-        <child link="chassis" />
-        <origin xyz="-0.1 0 0" rpy="0 0 0" />
-    </joint>
     <joint name="caster_wheel_joint" type="fixed">
         <parent link="chassis" />
@@ -76,5 +77,5 @@
             <origin xyz="0 0 0" rpy="0 0 0" />
             <geometry>
-                <sphere radius="0.1" />
+                <sphere radius="0.035" />
             </geometry>
             <material name="orange" />
@@ -86,5 +87,5 @@
             </geometry>
         </collision>
-        <xacro:sphere_inertia m="0.1" r="0.1" o_xyz="0 0 0" o_rpy="0 0 0" />
+        <xacro:sphere_inertia m="0.1" r="0.035" o_xyz="0 0 0" o_rpy="0 0 0" />
     </link>
 </robot>
