Commit message: Lidar inluded and updated.

File: description/camera.xacro (robot description, xacro)
@@ -1,14 +1,14 @@
 <?xml version="1.0"?>
 <robot xmlns:xacro="http://www.ros.org/wiki/xacro">
-    <joint name="laser_joint" type="fixed">
+    <joint name="camera_joint" type="fixed">
         <parent link="chassis" />
-        <child link="laser_frame" />
-        <origin xyz="0.2 0 0.1" rpy="0 0 0" />
+        <child link="camera_link" />
+        <origin xyz="0.305 0 0.07" rpy="0 0 0" />
     </joint>
-    <link name="laser_frame">
+    <link name="camera_link">
         <visual>
-            <origin xyz="0 0 0.025" rpy="0 0 0" />
+            <origin xyz="0 0 0" rpy="0 0 0" />
             <geometry>
-                <cylinder length="0.05" radius="0.05" />
+                <box size="0.01 0.03 0.03" />
             </geometry>
             <material name="red" />
@@ -17,16 +17,25 @@
             <origin xyz="0 0 0" rpy="0 0 0" />
             <geometry>
-                <cylinder length="0.05" radius="0.05" />
+                <box size="0.01 0.03 0.03" />
             </geometry>
         </collision>
-        <xacro:cylinder_inertia m="0.1" r="0.05" l="0.05" o_xyz="0 0 0" o_rpy="0 0 0" />
+        <xacro:box_inertia m="0.1" x="0.01" y="0.03" z="0.03" o_xyz="0.15 0 0.05" o_rpy="0 0 0" />
     </link>
-    <gazebo reference="laser_frame">
-        <sensor name="laser" type="lidar">
+    <joint name="camera_optical_joint" type="fixed">
+        <parent link="camera_link" />
+        <child link="camera_link_optical" />
+        <origin xyz="0 0 0" rpy="${-pi/2} 0 ${-pi/2}" />
+    </joint>
+    <link name="camera_link_optical">
+        <!-- This link is used to define the optical frame of the camera -->
+    </link>
+    <gazebo reference="camera_link">
+    </gazebo>
+</robot>
+<!-- <sensor name="camera" type="depth_camera">
             <pose>0 0 0 0 0 0</pose>
             <update_rate>10</update_rate>
             <visualize>true</visualize>
             <always_on>true</always_on>
-            <!-- Tell gz-sim where to publish -->
             <topic>/model/wally_boxxy/scan</topic>
             <ray>
@@ -50,5 +59,3 @@
                 </noise>
             </ray>
-        </sensor>
-    </gazebo>
-</robot>
+        </sensor> -->

File: description/gazebo_control.xacro (robot description, xacro)
@@ -1,21 +1,5 @@
 <?xml version="1.0"?>
 <robot xmlns:xacro="http://www.ros.org/wiki/xacro">
-    <!-- <gazebo>
-        <plugin name="diff_drive" filename="libgazebo_ros_diff_drive.so">
-            <left_joint>left_wheel_joint</left_joint>
-            <right_joint>right_wheel_joint</right_joint>
-            <wheel_separation>0.45</wheel_separation>
-            <wheel_radius>0.055</wheel_radius>
-            <use_ros_control>true</use_ros_control>
-            <max_wheel_torque>5.0</max_wheel_torque>
-            <max_wheel_acceleration>10.0</max_wheel_acceleration>
-            <odometry_frame>odom</odometry_frame>
-            <robot_base_frame>base_link</robot_base_frame>
-            <publish_odom>true</publish_odom>
-            <publish_odom_tf>true</publish_odom_tf>
-            <publish_wheel_tf>true</publish_wheel_tf>
-        </plugin>
-    </gazebo> -->
-    <gazebo reference="castor_wheel_link">
+    <gazebo reference="castor_wheel">
         <mu1 value="0.1" />
         <mu2 value="0.1" />
@@ -27,5 +11,5 @@
             <left_joint>left_wheel_joint</left_joint>
             <right_joint>right_wheel_joint</right_joint>
-            <wheel_separation>0.44</wheel_separation>
+            <wheel_separation>0.34</wheel_separation>
             <wheel_radius>0.055</wheel_radius>
             <frame_id>odom</frame_id>

File: description/robot.urdf.xacro (robot description, xacro)
@@ -1,7 +1,8 @@
 <?xml version="1.0"?>
-<robot xmlns:xacro="http://www.ros.org/wiki/xacro"  name="robot">
+<robot xmlns:xacro="http://www.ros.org/wiki/xacro"  name="wally_boxxy">
     <xacro:include filename="$(find wally_boxxy)/description/common_propreties.xacro" />
     <xacro:include filename="$(find wally_boxxy)/description/robot_core.xacro" />
     <xacro:include filename="$(find wally_boxxy)/description/gazebo_control.xacro" />
-    <xacro:include filename="$(find wally_boxxy)/description/lidar.xacro" />
+    <!-- <xacro:include filename="$(find wally_boxxy)/description/lidar.xacro" /> -->
+    <xacro:include filename="$(find wally_boxxy)/description/camera.xacro" />
 </robot>

File: description/robot_core.xacro (robot description, xacro)
@@ -6,26 +6,26 @@
         <parent link="base_link" />
         <child link="chassis" />
-        <origin xyz="-0.3 0 0.035" rpy="0 0 0" />
+        <origin xyz="-0.15 0 0.035" rpy="0 0 0" />
     </joint>
     <link name="chassis">
         <visual>
-            <origin xyz="0.3 0 0.1" rpy="0 0 0" />
+            <origin xyz="0.15 0 0.05" rpy="0 0 0" />
             <geometry>
-                <box size="0.6 0.4 0.2" />
+                <box size="0.3 0.2 0.1" />
             </geometry>
             <material name="blue" />
         </visual>
         <collision>
-            <origin xyz="0.3 0 0.1" rpy="0 0 0" />
+            <origin xyz="0.15 0 0.05" rpy="0 0 0" />
             <geometry>
-                <box size="0.6 0.4 0.2" />
+                <box size="0.3 0.2 0.1" />
             </geometry>
         </collision>
-        <xacro:box_inertia m="5" x="0.6" y="0.4" z="0.2" o_xyz="0.3 0 0.1" o_rpy="0 0 0" />
+        <xacro:box_inertia m="5" x="0.3" y="0.2" z="0.1" o_xyz="0.15 0 0.05" o_rpy="0 0 0" />
     </link>
     <joint name="left_wheel_joint" type="continuous">
         <parent link="chassis" />
         <child link="left_wheel" />
-        <origin xyz="0.1 0.22 0.02" rpy="-${pi/2} 0 0" />
+        <origin xyz="0.06 0.12 0.02" rpy="-${pi/2} 0 0" />
         <axis xyz="0 0 1" />
     </joint>
@@ -49,5 +49,5 @@
         <parent link="chassis" />
         <child link="right_wheel" />
-        <origin xyz="0.1 -0.22 0.02" rpy="${pi/2} 0 0" />
+        <origin xyz="0.06 -0.12 0.02" rpy="${pi/2} 0 0" />
         <axis xyz="0 0 1" />
     </joint>
@@ -71,5 +71,5 @@
         <parent link="chassis" />
         <child link="caster_wheel" />
-        <origin xyz="0.5 0 0" rpy="0 0 0" />
+        <origin xyz="0.25 0 0" rpy="0 0 0" />
     </joint>
     <link name="caster_wheel">
@@ -84,8 +84,59 @@
             <origin xyz="0 0 0" rpy="0 0 0" />
             <geometry>
-                <sphere radius="0.1" />
+                <sphere radius="0.035" />
             </geometry>
         </collision>
         <xacro:sphere_inertia m="0.1" r="0.035" o_xyz="0 0 0" o_rpy="0 0 0" />
     </link>
+    <joint name="laser_joint" type="fixed">
+        <parent link="chassis" />
+        <child link="laser_frame" />
+        <origin xyz="0.2 0 0.1" rpy="0 0 0" />
+    </joint>
+    <link name="laser_frame">
+        <visual>
+            <origin xyz="0 0 0.025" rpy="0 0 0" />
+            <geometry>
+                <cylinder length="0.05" radius="0.05" />
+            </geometry>
+            <material name="red" />
+        </visual>
+        <collision>
+            <origin xyz="0 0 0" rpy="0 0 0" />
+            <geometry>
+                <cylinder length="0.05" radius="0.05" />
+            </geometry>
+        </collision>
+        <xacro:cylinder_inertia m="0.1" r="0.05" l="0.05" o_xyz="0 0 0" o_rpy="0 0 0" />
+    </link>
+    <gazebo reference="laser_frame">
+        <sensor name="laser" type="lidar">
+            <pose>0 0 0 0 0 0</pose>
+            <update_rate>10</update_rate>
+            <visualize>true</visualize>
+            <always_on>true</always_on>
+            <!-- Tell gz-sim where to publish -->
+            <topic>/model/wally_boxxy/scan</topic>
+            <ray>
+                <scan>
+                    <horizontal>
+                    <samples>360</samples>
+                    <resolution>1</resolution>
+                    <min_angle>-3.14159</min_angle>
+                    <max_angle>3.14159</max_angle>
+                    </horizontal>
+                </scan>
+                <range>
+                    <min>0.3</min>
+                    <max>12</max>
+                    <resolution>0.01</resolution>
+                </range>
+                <noise>
+                    <type>gaussian</type>
+                    <mean>0.0</mean>
+                    <stddev>0.01</stddev>
+                </noise>
+            </ray>
+        </sensor>
+    </gazebo>
 </robot>
